File: Palm_IIIc_CCFL_replacement.kicad_pcb (KiCad board)
At the start: 2 copper layers, 74.5 x 9 mm, 52 parts

Commit message: Add additional supports to PCB
Parts:
- added 1: , , F.Cu at (116.4, 102.0)
- added 10: , , F.Cu at (159.6, 102.0)
- added 2: , , F.Cu at (115.5, 102.0)
- added 3: , , F.Cu at (127.4, 102.0)
- added 4: , , F.Cu at (126.5, 102.0)
- added 5: , , F.Cu at (138.4, 102.0)
- added 6: , , F.Cu at (137.6, 102.0)
- added 7: , , F.Cu at (149.4, 102.0)
- added 8: , , F.Cu at (148.6, 102.0)
- added 9: , , F.Cu at (160.4, 102.0)
- added ?: , , F.Cu at (105.4, 102.0)
- added ?: , , F.Cu at (104.5, 102.0)
- added REF**: Perforation_0.4mm, Perforation:Perforation_0.4mm, F.Cu at (103.7, 102.0)
- added REF**1: Perforation_0.4mm, Perforation:Perforation_0.4mm, F.Cu at (114.7, 102.0)
- added REF**2: Perforation_0.4mm, Perforation:Perforation_0.4mm, F.Cu at (125.7, 102.0)
- added REF**3: Perforation_0.4mm, Perforation:Perforation_0.4mm, F.Cu at (136.7, 102.0)
- added REF**4: Perforation_0.4mm, Perforation:Perforation_0.4mm, F.Cu at (147.7, 102.0)
- added REF**5: Perforation_0.4mm, Perforation:Perforation_0.4mm, F.Cu at (158.7, 102.0)
Other:
- outline, holes or cut-outs redrawn
