File: led.kicad_sch (KiCad schematic)
At the start: 2 parts

Commit message: Add README
Parts:
- R1: value 330R -> 220R
Changed lines of the file:
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@@
     (in_bom yes) (on_board yes) (fields_autoplaced)
     (property "Reference" "R1" (id 0) (at 130.81 88.2736 90))
-    (property "Value" "330R" (id 1) (at 130.81 90.8105 90))
+    (property "Value" "220R" (id 1) (at 130.81 90.8105 90))
     (property "Footprint" "Resistor_SMD:R_0402_1005Metric" (id 2) (at 130.81 92.71 0)
       (effects (font (size 1.27 1.27)) hide)
